Commit message: kamera + AprilTag: kafa kameralarından /luna/dock/tag, kafa dönüşü telafili
- core/dock_tag.py: etiketin base_link konumu → (offset, ağız–burun mesafesi), iki kamera birleştirme; R02 CAD geometrisi
- core/frames.py (URDF zinciri), camera_model.py (B0630 720p), tag36h11.py, tag_scene.py (sentetik görüntü)
- dock_tag_node: apriltag_ros tespitleri → TF → /luna/dock/tag; bloklamayan TF bekleme kuyruğu
- sim_camera_node + tags:=mock|sim|usb; mock gerçek pozu /luna/mock/truth'a yayımlar
- head_node /joint_states yayımlar (TF'de kafa/kamera zinciri yoktu); URDF kameraları R06 modeline, optik çerçeveler
- usb_cam (1280×720 MJPG, 15 fps), apriltag_ros (tag36h11 ID 0, 48 mm), nominal camera_info, baskı SVG'si
- Fast DDS 4 MB SHM profili: 720p görüntüler süreçler arası 2.4 s'ye kadar takılıyordu
- 22 yeni test (63); sentetik tarama 272/272 (≤2.0 m), tags:=sim tam yığın CHARGING (düz, kafa +30°, 20° dönük)

Co-Authored-By: Claude Opus 5.5 <noreply@anthropic.com>

File: luna_ws/src/luna_robot/urdf/luna.urdf (robot description, URDF)
Before this commit: robot luna, 11 links, 10 joints
Links:
- added link camera_left_optical_frame
- added link camera_right_optical_frame
Joints:
- added joint camera_left_optical_joint: type fixed, parent camera_left_link, child camera_left_optical_frame, origin rpy=-1.5707963267948966 0 -1.5707963267948966
- added joint camera_right_optical_joint: type fixed, parent camera_right_link, child camera_right_optical_frame, origin rpy=-1.5707963267948966 0 -1.5707963267948966
- joint camera_left_joint: origin xyz=0.040 0.062 0.010 -> xyz=0.064 0.062 0.010
- joint camera_right_joint: origin xyz=0.040 -0.062 0.010 -> xyz=0.064 -0.062 0.010

Commit message: WIP engel-algilama: 2.5B simülatör çekirdeği, URDF ToF/OAK-D çerçeveleri
- urdf: oakd_link/oakd_optical_frame (geçici poz, R08 bekleniyor), tof_fl/fr/bl/br (R07 FOV koni tepeleri, düz ileri/geri)
- core/robot_model.py: URDF'ten sensör pozları (tek yer)
- core/sim2d.py: Block/Cylinder yükseklik bantlı engeller, LiDAR düzlem kesiti, ToF koni ışınları (zemin dahil),
  robot yükseklik bantları ile temas (tampon / kaza) günlüğü
- core/sim_worlds.py: room/toy/table/chair/dock/door dünyaları
- core/depth_camera.py: numpy OAK-D Lite derinlik raycast (Docker'da denenmedi)
- core/tof.py: köşe ToF -> Range dönüşümü
Mevcut 204 birim testi Mac'te geçiyor (7 atlandı). Düğümler, Nav2, launch, senaryolar ve yeni testler henüz yok.

Co-Authored-By: Claude Opus 5.5 <noreply@anthropic.com>

File: luna_ws/src/luna_robot/urdf/luna.urdf (robot description, URDF)
Before this commit: robot luna, 13 links, 12 joints
Links:
- added link oakd_link
- added link oakd_optical_frame
- added link tof_bl
- added link tof_br
- added link tof_fl
- added link tof_fr
Joints:
- added joint oakd_joint: type fixed, parent base_link, child oakd_link, origin xyz=0.105 0 0.365 rpy=0 0.2617993877991494 0
- added joint oakd_optical_joint: type fixed, parent oakd_link, child oakd_optical_frame, origin rpy=-1.5707963267948966 0 -1.5707963267948966
- added joint tof_bl_joint: type fixed, parent base_link, child tof_bl, origin xyz=-0.16888 0.09355 0.101 rpy=0 0 3.141592653589793
- added joint tof_br_joint: type fixed, parent base_link, child tof_br, origin xyz=-0.16888 -0.09355 0.101 rpy=0 0 3.141592653589793
- added joint tof_fl_joint: type fixed, parent base_link, child tof_fl, origin xyz=0.16888 0.09355 0.101
- added joint tof_fr_joint: type fixed, parent base_link, child tof_fr, origin xyz=0.16888 -0.09355 0.101

Commit message: WIP engel-algilama: R08 sensör pozları (LiDAR Z0.5898 yaw −90°, depthai optik çerçeveleri, tof_down)
Co-Authored-By: Claude Opus 5.5 <noreply@anthropic.com>

File: luna_ws/src/luna_robot/urdf/luna.urdf (robot description, URDF)
Before this commit: robot luna, 19 links, 18 joints
Links:
- removed link oakd_optical_frame
- added link oak_left_camera_optical_frame
- added link oak_rgb_camera_optical_frame
- added link oak_right_camera_optical_frame
- added link tof_down_bl
- added link tof_down_br
- added link tof_down_fl
- added link tof_down_fr
Joints:
- removed joint oakd_joint
- removed joint oakd_optical_joint
- added joint oak_left_camera_optical_frame_joint: type fixed, parent base_link, child oak_left_camera_optical_frame, origin xyz=0.1115 0.0375 0.3685 rpy=-1.8326 -0.0000 -1.5708
- added joint oak_rgb_camera_optical_frame_joint: type fixed, parent base_link, child oak_rgb_camera_optical_frame, origin xyz=0.1130 0.0000 0.3681 rpy=-1.8326 -0.0000 -1.5708
- added joint oak_right_camera_optical_frame_joint: type fixed, parent base_link, child oak_right_camera_optical_frame, origin xyz=0.1115 -0.0375 0.3685 rpy=-1.8326 -0.0000 -1.5708
- added joint oakd_link_joint: type fixed, parent base_link, child oakd_link, origin xyz=0.1050 0.0000 0.3650 rpy=-0.0000 0.2618 -0.0000
- added joint tof_down_bl_joint: type fixed, parent base_link, child tof_down_bl, origin xyz=-0.1360 0.1085 0.0532 rpy=-0.0000 1.5708 0.0000
- added joint tof_down_br_joint: type fixed, parent base_link, child tof_down_br, origin xyz=-0.1360 -0.1085 0.0532 rpy=-0.0000 1.5708 0.0000
- added joint tof_down_fl_joint: type fixed, parent base_link, child tof_down_fl, origin xyz=0.1360 0.1085 0.0532 rpy=-0.0000 1.5708 0.0000
- added joint tof_down_fr_joint: type fixed, parent base_link, child tof_down_fr, origin xyz=0.1360 -0.1085 0.0532 rpy=-0.0000 1.5708 0.0000
- joint laser_joint: origin xyz=-0.070 0 0.580 -> xyz=-0.0700 0.0000 0.5898 rpy=0.0000 -0.0000 -1.5708
- joint tof_bl_joint: origin xyz=-0.16888 0.09355 0.101 rpy=0 0 3.141592653589793 -> xyz=-0.1689 0.0935 0.1010 rpy=0.0000 -0.0000 3.1416
- joint tof_br_joint: origin xyz=-0.16888 -0.09355 0.101 rpy=0 0 3.141592653589793 -> xyz=-0.1689 -0.0935 0.1010 rpy=0.0000 -0.0000 3.1416
- joint tof_fl_joint: origin xyz=0.16888 0.09355 0.101 -> xyz=0.1689 0.0935 0.1010 rpy=-0.0000 -0.0000 0.0000
- joint tof_fr_joint: origin xyz=0.16888 -0.09355 0.101 -> xyz=0.1689 -0.0935 0.1010 rpy=-0.0000 -0.0000 0.0000

Commit message: R2: sabit ekranlı kafa, tepede LiDAR, diferansiyel sürüş; Türkiye'de bulunan parçalar
Tasarım (docs/TASARIM_R2.md) ve Türkiye malzeme listesi (docs/MALZEME_LISTESI.md):
- Yüz kafadaki 5,5" AMOLED dokunmatik ekranda; telefon gerekmiyor. Kafa sabit,
  ekranın üstünde tek yüz kamerası (Pi Camera v2), RPLIDAR C1 kafanın tepesinde.
- Ø 360 mm yuvarlak gövde, tam saran tampon halkası; ortada iki tahrikli teker
  (Pololu 37D 70:1), önde ve arkada birer sarhoş teker.
- Jetson Orin NX 16 GB, Orbbec Gemini 336, ReSpeaker Mic Array v2.0,
  4S2P LiFePO4 + Daly BMS, VL53L1X uçurum sensörleri.

Yazılım:
- URDF, kinematik (jiroskop füzyonu), dikkat (gövde dönüşü), yüz takibi,
  ReSpeaker ve gizlilik sürgüsü, Gemini derinlik ve renk kamerası, dock etiketi,
  2.5B simülatör (yuvarlak gövde, R2 dock'u), Nav2 dairesel ayak izi.
- Kafa servoları ve kafa düğümü kaldırıldı.
- Ekran yüzü: web/face-core.js, face.js, face.html; tools/kiosk.sh.
- Firmware: servolar çıktı; Daly BMS ayrıştırıcısı, VL53L1X zemin sensörleri,
  4480 CPR enkoder.
- Docker: JetPack 6 (l4t-jetpack r36.4.0), ROS apt'tan, OrbbecSDK_ROS2 v2.9.3,
  whisper.cpp (CUDA), Piper.

Doğrulama (README_TR.md, "R2 doğrulama"):
- Python 311/311; colcon test 311/311; web 21/21.
- Firmware host 19 test, 188 kontrol; Teensy derlemesi 0 uyarı.
- Kamerayla dock: gerçek apriltag_ros ile CHARGING.
- Haritalama 17/17, yerelleştirme 12/12.
- Parkurlar: toy, table, chair, door, door70 geçti; door60 2 koşunun 1'inde
  geçti; dock yolundaki eşyalar parkuru geçmedi (açık).
Gerçek donanımda denenmedi.

Co-Authored-By: Claude Opus 5.5 <noreply@anthropic.com>
Claude-Session: https://claude.ai/code/session_01KTiQHC9XsfxLZy6JEysTYw

File: luna_ws/src/luna_robot/urdf/luna.urdf (robot description, URDF)
Before this commit: robot luna, 25 links, 24 joints
Links:
- removed link camera_left_link
- removed link camera_left_optical_frame
- removed link camera_right_link
- removed link camera_right_optical_frame
- removed link head_pan_link
- removed link head_tilt_link
- removed link oak_left_camera_optical_frame
- removed link oak_rgb_camera_optical_frame
- removed link oak_right_camera_optical_frame
- removed link oakd_link
- removed link track_left
- removed link track_right
- added link camera_color_optical_frame
- added link camera_depth_optical_frame
- added link camera_imu_frame
- added link camera_link
- added link caster_front
- added link caster_rear
- added link face_camera_link
- added link face_camera_optical_frame
- added link head_link; visual box size=0.120 0.220 0.160
- added link mic_array
- added link wheel_left; visual cylinder length=0.010 radius=0.040
- added link wheel_right; visual cylinder length=0.010 radius=0.040
- link base_link: geometry visual cylinder length=0.330 radius=0.180
Joints:
- removed joint camera_left_joint
- removed joint camera_left_optical_joint
- removed joint camera_right_joint
- removed joint camera_right_optical_joint
- removed joint head_pan
- removed joint head_tilt
- removed joint oak_left_camera_optical_frame_joint
- removed joint oak_rgb_camera_optical_frame_joint
- removed joint oak_right_camera_optical_frame_joint
- removed joint oakd_link_joint
- removed joint track_left_joint
- removed joint track_right_joint
- added joint camera_color_optical_joint: type fixed, parent camera_link, child camera_color_optical_frame, origin xyz=0 0.0080 0 rpy=-1.5707963267948966 0 -1.5707963267948966
- added joint camera_depth_optical_joint: type fixed, parent camera_link, child camera_depth_optical_frame, origin xyz=0 0 0 rpy=-1.5707963267948966 0 -1.5707963267948966
- added joint camera_imu_joint: type fixed, parent camera_link, child camera_imu_frame
- added joint camera_link_joint: type fixed, parent base_link, child camera_link, origin xyz=0.1650 0.0000 0.2700 rpy=0.0000 0.2618 0.0000
- added joint caster_front_joint: type fixed, parent base_link, child caster_front, origin xyz=0.110 0 0.0127
- added joint caster_rear_joint: type fixed, parent base_link, child caster_rear, origin xyz=-0.110 0 0.0127
- added joint face_camera_joint: type fixed, parent head_link, child face_camera_link, origin xyz=0.072 0 0.145 rpy=0 -0.2094 0
- added joint face_camera_optical_joint: type fixed, parent face_camera_link, child face_camera_optical_frame, origin rpy=-1.5707963267948966 0 -1.5707963267948966
- added joint head_joint: type fixed, parent base_link, child head_link, origin xyz=0 0 0.360
- added joint mic_array_joint: type fixed, parent base_link, child mic_array, origin xyz=-0.0700 0 0.3480
- added joint wheel_left_joint: type fixed, parent base_link, child wheel_left, origin xyz=0 0.150 0.040
- added joint wheel_right_joint: type fixed, parent base_link, child wheel_right, origin xyz=0 -0.150 0.040
- joint dock_contact_joint: origin xyz=0.159 0 0.102 -> xyz=0.060 0.060 0.015
- joint face_display_joint: origin xyz=0.115 0 0.256 rpy=0 -0.1666 0 -> xyz=0.072 0 0.080 rpy=0 -0.1396 0; parent base_link -> head_link
- joint laser_joint: origin xyz=-0.0700 0.0000 0.5898 rpy=0.0000 -0.0000 -1.5708 -> xyz=0.0000 0.0000 0.5498 rpy=0.0000 -0.0000 -1.5708
- joint tof_bl_joint: origin xyz=-0.1689 0.0935 0.1010 rpy=0.0000 -0.0000 3.1416 -> xyz=-0.1434 0.1004 0.1000 rpy=0 0 2.6180
- joint tof_br_joint: origin xyz=-0.1689 -0.0935 0.1010 rpy=0.0000 -0.0000 3.1416 -> xyz=-0.1434 -0.1004 0.1000 rpy=0 0 -2.6180
- joint tof_down_bl_joint: origin xyz=-0.1360 0.1085 0.0532 rpy=-0.0000 1.5708 0.0000 -> xyz=-0.1540 0.0720 0.0600 rpy=0 1.5708 0
- joint tof_down_br_joint: origin xyz=-0.1360 -0.1085 0.0532 rpy=-0.0000 1.5708 0.0000 -> xyz=-0.1540 -0.0720 0.0600 rpy=0 1.5708 0
- joint tof_down_fl_joint: origin xyz=0.1360 0.1085 0.0532 rpy=-0.0000 1.5708 0.0000 -> xyz=0.1540 0.0720 0.0600 rpy=0 1.5708 0
- joint tof_down_fr_joint: origin xyz=0.1360 -0.1085 0.0532 rpy=-0.0000 1.5708 0.0000 -> xyz=0.1540 -0.0720 0.0600 rpy=0 1.5708 0
- joint tof_fl_joint: origin xyz=0.1689 0.0935 0.1010 rpy=-0.0000 -0.0000 0.0000 -> xyz=0.1434 0.1004 0.1000 rpy=0 0 0.5236
- joint tof_fr_joint: origin xyz=0.1689 -0.0935 0.1010 rpy=-0.0000 -0.0000 0.0000 -> xyz=0.1434 -0.1004 0.1000 rpy=0 0 -0.5236

Commit message: Köşe ToF'ları düz baksın: eğik yan duvar dar geçitleri kapatıyordu
İlk simülatör koşularında dock yolundaki eşyalar parkuru başarısız oldu
(RPP ayakkabı kutusunun yanında "collision ahead" deyip takıldı, Nav2
240 s'de vazgeçti). 60 cm kapı da 2 koşunun 1'inde geçemedi.

Nedeni: köşe ToF'ları 30° dışa bakıyordu ve tof_range_node her okumayı
koninin bütün genişliğinde bir yay olarak haritaya işliyor. Yan duvarı eğik
gören koni, yayın uçlarını gerçek yüzeyin 14-20 cm önüne düşürüyordu; 68 cm'lik
geçidin ortasında robot merkezine ~2 cm kalıyordu. Ölçüm simülatörün kendi ToF
modeliyle yapıldı.

Düzeltme: ToF'lar düz ileri/geri bakıyor. Yuvarlak gövde yerinde dönerken
yanlara taşmadığı için yan kapsama gerekmiyor.

Sonrasında bütün senaryolar yeniden koşuldu, 11/11 geçti:
- haritalama 17/17, yerelleştirme 12/12
- dock yolu 2/2, 60 cm kapı 2/2
- 70 cm kapı, toy, table, chair, kapalı kapı
- temas 0

Kalan risk: dock yolunda 10 cm'lik kutuya 5-7 cm açıklık.
README ve tasarım belgesi bu sonuçlarla güncellendi.

Co-Authored-By: Claude Opus 5.5 <noreply@anthropic.com>
Claude-Session: https://claude.ai/code/session_01KTiQHC9XsfxLZy6JEysTYw

File: luna_ws/src/luna_robot/urdf/luna.urdf (robot description, URDF)
Before this commit: robot luna, 25 links, 24 joints
Joints:
- joint tof_bl_joint: origin xyz=-0.1434 0.1004 0.1000 rpy=0 0 2.6180 -> xyz=-0.1434 0.1004 0.1000 rpy=0 0 3.1416
- joint tof_br_joint: origin xyz=-0.1434 -0.1004 0.1000 rpy=0 0 -2.6180 -> xyz=-0.1434 -0.1004 0.1000 rpy=0 0 3.1416
- joint tof_fl_joint: origin xyz=0.1434 0.1004 0.1000 rpy=0 0 0.5236 -> xyz=0.1434 0.1004 0.1000 rpy=0 0 0
- joint tof_fr_joint: origin xyz=0.1434 -0.1004 0.1000 rpy=0 0 -0.5236 -> xyz=0.1434 -0.1004 0.1000 rpy=0 0 0
